Commit message: Final commit of EECS498 Lab 4. Hokuyo LIDAR meshes not working (?).

File: urdf/robot.xacro (robot description, xacro)
@@ -24,5 +24,5 @@
 <xacro:laser name="laser_vert_top_right" parent="base" xyz="0.2978 -0.1450 1.8451" rpy="-1.1760 0.6313 -1.9377" meshes="package://gazebo_plugins/test/multi_robot_scenario/meshes/laser" />
 <xacro:laser name="laser_vert_top_left" parent="base" xyz="0.2997 0.1531 1.8443" rpy="1.1780 0.6198 1.9560" meshes="package://gazebo_plugins/test/multi_robot_scenario/meshes/laser" />
-<VLP-16 parent="base" name="laser_horiz" topic="laser_horiz/packets" hz="10" samples="440" gpu="false">
+<VLP-16 parent="base" name="laser_horiz" topic="laser_horiz/packets" hz="10" samples="440" gpu="false" >
 <origin xyz="0.2325416305773505 -0.0001380069427607134 1.920122926231907" rpy="-0.0012068 0.114646 -0.0015308" />
 </VLP-16>

File: urdf/urdf_from_xacro.urdf (robot description, URDF)
Before this commit: robot robot_description, 6 links, 5 joints
Links:
- removed link base_link
- added link base; collision box size=0.94 0.78 1.98; visual box size=0.94 0.78 1.98
- added link laser_horiz_base_link, mass 0.83; collision cylinder length=0.0717 radius=0.0516; visual mesh filename=package://velodyne_description/meshes/VLP16_base_1.dae
- added link wheel_center; collision cylinder length=0.05 radius=0.15; visual cylinder length=0.05 radius=0.15
- added link wheel_right; collision cylinder length=0.05 radius=0.2; visual cylinder length=0.05 radius=0.2
- link laser_horiz: mass None -> 0.01; geometry visual mesh filename=package://velodyne_description/meshes/VLP16_scan.dae
- link laser_vert_bottom: mass None -> 1e-5; geometry collision box size=0.1 0.1 0.1; visual mesh filename=package://gazebo_plugins/test/multi_robot_scenario/meshes/l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
- link laser_vert_top_left: mass None -> 1e-5; geometry collision box size=0.1 0.1 0.1; visual mesh filename=package://gazebo_plugins/test/multi_robot_scenario/meshes/l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
- link laser_vert_top_right: mass None -> 1e-5; geometry collision box size=0.1 0.1 0.1; visual mesh filename=package://gazebo_plugins/test/multi_robot_scenario/meshes/l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
Joints:
- removed joint base_to_horiz
- removed joint base_to_vert_bottom
- removed joint base_to_vert_top_left
- removed joint base_to_vert_top_right
- added joint base_laser_vert_bottom_joint: type fixed, parent base, child laser_vert_bottom, origin xyz=0.3157894464801903 -0.002068548615034871 0.5099999434059285 rpy=3.1354753 -1.3045001 0.0024658, axis 0 0 1
- added joint base_laser_vert_top_left_joint: type fixed, parent base, child laser_vert_top_left, origin xyz=0.2997 0.1531 1.8443 rpy=1.1780 0.6198 1.9560, axis 0 0 1
- added joint base_laser_vert_top_right_joint: type fixed, parent base, child laser_vert_top_right, origin xyz=0.2978 -0.1450 1.8451 rpy=-1.1760 0.6313 -1.9377, axis 0 0 1
- added joint base_to_wheel_center: type continuous, parent base, child wheel_center, origin xyz=0 0 0, limit effort=1 velocity=1
- added joint base_to_wheel_right: type continuous, parent base, child wheel_right, origin xyz=0 0 0, limit effort=1 velocity=1
- added joint laser_horiz_base_mount_joint: type fixed, parent base, child laser_horiz_base_link, origin xyz=0.2325416305773505 -0.0001380069427607134 1.920122926231907 rpy=-0.0012068 0.114646 -0.0015308
- added joint laser_horiz_base_scan_joint: type fixed, parent laser_horiz_base_link, child laser_horiz, origin xyz=0 0 0.0377 rpy=0 0 0
- joint base_to_wheel_left: limit effort= velocity= -> effort=1 velocity=1; parent base_link -> base; type fixed -> continuous

Commit message: Final commit of EECS498 Lab 4. Hokuyo LIDAR meshes not working (?).

File: urdf/robot.xacro (robot description, xacro)
@@ -21,5 +21,5 @@
     </collision>
   </link>
-<xacro:laser name="laser_vert_bottom" parent="base" xyz="0.3157894464801903 -0.002068548615034871 0.5099999434059285" rpy="3.1354753 -1.3045001 0.0024658" meshes="package://gazebo_plugins/test/multi_robot_scenario/meshes/laser" />
+<xacro:laser name="laser_vert_bottom" parent="base" xyz="0.3157 -0.0021 0.5099" rpy="3.1354 -1.3045 0.0025" meshes="package://gazebo_plugins/test/multi_robot_scenario/meshes/laser" />
 <xacro:laser name="laser_vert_top_right" parent="base" xyz="0.2978 -0.1450 1.8451" rpy="-1.1760 0.6313 -1.9377" meshes="package://gazebo_plugins/test/multi_robot_scenario/meshes/laser" />
 <xacro:laser name="laser_vert_top_left" parent="base" xyz="0.2997 0.1531 1.8443" rpy="1.1780 0.6198 1.9560" meshes="package://gazebo_plugins/test/multi_robot_scenario/meshes/laser" />
@@ -129,26 +129,4 @@
 </xacro:macro>
 <xacro:wheelmaker suffix="left" reflect="1" />
-<xacro:macro name="wheelmaker" params="suffix reflect">
-	<link name="wheel_${suffix}">
-		<visual>
-			<geometry>
-				<cylinder radius="0.2" length="0.05" />
-			</geometry>
-			<origin xyz="-0.10 ${reflect*0.4} 0.0" rpy="${-pi/2} 0 0" />
-		</visual>
-		<collision>
-			<geometry>
-				<cylinder radius="0.2" length="0.05" />
-			</geometry>
-			<origin xyz="-0.10 ${reflect*0.4} 0.0" rpy="${-pi/2} 0 0" />
-		</collision>
-	</link>
-	<joint name="base_to_wheel_${suffix}" type="continuous">
-		<parent link="base" />
-		<child link="wheel_${suffix}" />
-		<origin xyz="0 0 0" />
-		<limit effort="1" velocity="1" />
-	</joint>
-</xacro:macro>
 <xacro:wheelmaker suffix="right" reflect="-1" />
 <xacro:macro name="wheelmaker" params="suffix reflect">
